File: plant_controller/plant_controller.kicad_pcb (KiCad board)
At the start: 2 copper layers, 41.9 x 71.1 mm, 13 parts, among them J1 Conn_01x03_Pin, J2 Conn_01x03_Pin, J3 Conn_01x19_Socket, J4 Conn_01x19_Socket, J5 Conn_01x04_Socket, SW1 RotaryEncoder, SW2 RotaryEncoder

Commit message: added small plant controller project
Parts:
- added R5: 47K, Resistor_SMD:R_1206_3216Metric, B.Cu at (79.0, 55.6)
- added R6: 47K, Resistor_SMD:R_1206_3216Metric, B.Cu at (81.5, 55.6)
Routing:
- net GND: track 14.9 -> 37.6 mm
- net Net-(J1-Pin_3): track 33.6 -> 42.3 mm
- net Net-(J2-Pin_3): track 8.67 -> 13.7 mm
Other:
- board text added: "- +"
