File: plant_controller/plant_controller.kicad_sch (KiCad schematic)
At the start: 13 parts, among them J1 Conn_01x03_Pin, J2 Conn_01x03_Pin, J3 Conn_01x19_Socket, J4 Conn_01x19_Socket, J5 Conn_01x04_Socket, SW1 RotaryEncoder, SW2 RotaryEncoder

Commit message: added small plant controller project
Parts:
- added R5, R6: 47K, Resistor_SMD:R_1206_3216Metric, symbol Device:R
Connections:
- net GND: now also R5.2, R6.2
- net at J1.3 (Pin_3), J3.6 (Pin_6): now also R6.1
- net at J2.3 (Pin_3), J3.5 (Pin_5): now also R5.1
